Commit message: Minor changes

File: newbot_description/urdf/materials.xacro (robot description, xacro)
@@ -1,11 +1,11 @@
 <?xml version="1.0"?>
 <robot>
-	<material name="lightred">
-		<color rgba="0.5 0.0 0.0 1.0" />
+	<material name="top">
+		<color rgba="0.715 0.583 0.210 1.0"/>
 	</material>
-	<material name="red">
-		<color rgba="0.4 0.1 0.1 1.0"/>
+	<material name="body">
+		<color rgba="1.0 0.811 0.151 1.0"/>
 	</material>
-	<material name="darkgrey">
+	<material name="wheels">
 		<color rgba="0.117 0.117 0.117 1.0"/>
 	</material>

File: newbot_description/urdf/newbot.xacro (robot description, xacro)
@@ -15,5 +15,5 @@
      <box size="1.8 0.755 0.2" />
 	 </geometry>
-	 <material name="red" />
+	 <material name="body" />
 	</visual>
 	<collision>
@@ -45,5 +45,5 @@
           <cylinder length="0.26" radius="0.24"/>
         </geometry>
-        <material name="darkgrey" />
+        <material name="wheels" />
       </visual>
       <collision>
@@ -117,5 +117,5 @@
         <box size="0.5 0.25 0.1" />
       </geometry>
-      <material name="lightred"/>
+      <material name="top"/>
     </visual>
     <inertial>
@@ -143,5 +143,5 @@
   <box size="0.5 0.25 0.047" />
       </geometry>
-	<material name="lightred"/>
+	<material name="top"/>
     </visual>
     <inertial>
