Commit message: Slight updates

File: newbot_description/urdf/newbot.xacro (robot description, xacro)
@@ -26,14 +26,11 @@
 	 <origin xyz="0.0422171696051465 0.00189728780308063 -0.0378333807867307" rpy="0 0 0"/>
 	 <mass value="16.523"/>
-	 <inertia
-	  ixx="0.3136" ixy="-0.0008" ixz="0.0164"
-	  iyy="0.3922" iyz="-0.0009"
-	  izz="0.4485"/>
-	</inertial>
+	 <inertia ixx="0.3136" ixy="-0.0008" ixz="0.0164" iyy="0.3922" iyz="-0.0009" izz="0.4485"/>
+  </inertial>
 </link>
 <joint name="chasis_link_joint" type="fixed">
 	<origin xyz="0 0 0.375" rpy="0 0 0" />
 	<parent link="base_link"/>
-	<child link="chassis_link" />
+	<child link="chassis_link"/>
 </joint>
 <!--wheel-->
@@ -45,5 +42,5 @@
           <cylinder length="0.26" radius="0.24"/>
         </geometry>
-        <material name="wheels" />
+        <material name="wheels"/>
       </visual>
       <collision>
@@ -56,15 +53,12 @@
         <origin xyz="9.1812e-6 1.0274e-6 -4.4809e-6" rpy="0 0 0"/>
         <mass value="0.477"/>
-        <inertia
-          ixx="0.0013" ixy="0" ixz="0"
-          iyy="0.0024" iyz="0"
-          izz="0.0013"/>
+        <inertia ixx="0.0013" ixy="0" ixz="0" iyy="0.0024" iyz="0" izz="0.0013"/>
       </inertial>
 </link>
-	<gazebo reference="${prefix}_wheel_link">
-  	  <mu1>0.2</mu1>
- 	   <mu2>0.2</mu2>
-     	 <material>Gazebo/DarkGrey</material>
-	</gazebo>
+    <gazebo reference="${prefix}_wheel_link">
+      <mu1>0.2</mu1>
+      <mu2>0.2</mu2>
+      <material>Gazebo/DarkGrey</material>
+    </gazebo>
 	<joint name="${prefix}_wheel" type="continuous">
     	  <parent link="base_link"/>
@@ -73,5 +67,8 @@
    	   <axis xyz="0 1 0" />
 	</joint>
-    <!-- It's more straightforward for Gazebo to simulate as if there's an actuator per wheel. -->
+    <!--
+      Gazebo needs the following code
+      for each wheel to be actuatored
+    -->
 	<transmission name="${prefix}_wheel_trans">
     	  <type>transmission_interface/SimpleTransmission</type>
@@ -97,5 +94,5 @@
     <origin xyz="-0.70542 -0.51501 0.23923" rpy="0 0 0" />
   </xacro:wheel>
-<!-- end of wheel description -->>
+<!-- wheels section closed -->>
 <!-- laser base -->
   <joint name="camera_joint" type="fixed">
@@ -148,5 +145,5 @@
       <mass value="1e-5" />
       <origin xyz="-5.7094e-7 -8.9157e-6 0.1" rpy="0 0 0"/>
-      <inertia ixx="1e-6" ixy="0" ixz="0" iyy="1e-6" iyz="0" izz="1e-6" />
+      <inertia ixx="1e-6" ixy="0" ixz="0" iyy="1e-6" iyz="0" izz="1e-6"/>
     </inertial>
   </link>
